Commit message: Update simplfied description for successful gazebo run

File: ros/finalarm_simplified_description/urdf/finalarm_simplified.urdf.xacro (robot description, xacro)
@@ -1,43 +1,41 @@
-<?xml version="1.0"?>
+<?xml version="1.0" ?>
 <!-- Revolute-Revolute Manipulator -->
 <robot name="finalarm_simplified" xmlns:xacro="http://www.ros.org/wiki/xacro">
   <!-- Import all Gazebo-customization elements -->
-  <xacro:include filename="$(find finalarm_simplified_description)/urdf/finalarm_simplified.gazebo" />
+  <xacro:include
+    filename="$(find finalarm_simplified_description)/urdf/finalarm_simplified.gazebo"
+  />
   <link name="root">
     <visual>
       <origin xyz="0 0 0" rpy="0 0 0" />
       <geometry>
-        <box size = "0 0 0"/>
-      </geometry>
-    </visual>
-    <collision>
-      <origin xyz="0 0 0" rpy="0 0 0" />
-      <geometry>
-        <box size = "0 0 0"/>
+        <box size="0 0 0" />
+      </geometry>
+    </visual>
+    <collision>
+      <origin xyz="0 0 0" rpy="0 0 0" />
+      <geometry>
+        <box size="0 0 0" />
       </geometry>
     </collision>
   </link>
   <!-- Used for fixing robot to Gazebo 'base_link' -->
-  <link name="world"/>
+  <link name="world" />
   <joint name="connect_root_and_world" type="fixed">
-    <parent link="world"/>
-    <child link="root"/>
-    <axis xyz="0 0 0"/>
+    <parent link="world" />
+    <child link="root" />
+    <axis xyz="0 0 0" />
     <origin xyz="0 0 0" rpy="0 0 0" />
   </joint>
   <joint name="root_to_base_link" type="fixed">
-    <parent link="root"/>
-    <child link="base_link"/>
-    <axis xyz="0 0 0"/>
+    <parent link="root" />
+    <child link="base_link" />
+    <axis xyz="0 0 0" />
     <origin xyz="0 0 0" rpy="0 0 0" />
   </joint>
-  <link
-    name="base_link">
-    <inertial>
-      <origin
-        xyz="-0.0164 -8.67361737988404E-19 0.0311"
-        rpy="0 0 0" />
-      <mass
-        value="0.481547424" />
+  <link name="base_link">
+    <inertial>
+      <origin xyz="-0.0164 -8.67361737988404E-19 0.0311" rpy="0 0 0" />
+      <mass value="0.481547424" />
       <inertia
         ixx="0.00259388526"
@@ -46,38 +44,34 @@
         iyy="0.00279542583"
         iyz="-0.00000008121"
-        izz="0.00116940616" />
-    </inertial>
-    <visual>
-      <origin
-        xyz="0 0 0"
-        rpy="0 0 0" />
-      <geometry>
-        <mesh
-          filename="package://finalarm_simplified_description/meshes/base_link.STL" />
-      </geometry>
-      <material
-        name="">
-        <color
-          rgba="0.792156862745098 0.819607843137255 0.933333333333333 1" />
-      </material>
-    </visual>
-    <collision>
-      <origin
-        xyz="0 0 0"
-        rpy="0 0 0" />
-      <geometry>
-        <mesh
-          filename="package://finalarm_simplified_description/meshes/base_link.STL" />
-      </geometry>
-    </collision>
-  </link>
-  <link
-    name="link_2">
+        izz="0.00116940616"
+      />
+    </inertial>
+    <visual>
+      <origin xyz="0 0 0" rpy="0 0 0" />
+      <geometry>
+        <mesh
+          filename="package://finalarm_simplified_description/meshes/base_link.STL"
+        />
+      </geometry>
+      <material name="">
+        <color rgba="0.792156862745098 0.819607843137255 0.933333333333333 1" />
+      </material>
+    </visual>
+    <collision>
+      <origin xyz="0 0 0" rpy="0 0 0" />
+      <geometry>
+        <mesh
+          filename="package://finalarm_simplified_description/meshes/base_link.STL"
+        />
+      </geometry>
+    </collision>
+  </link>
+  <link name="link_2">
     <inertial>
       <origin
         xyz="-1.38777878078145E-17 -4.33680868994202E-18 -0.078375"
-        rpy="0 0 0" />
-      <mass
-        value="0.7142784" />
+        rpy="0 0 0"
+      />
+      <mass value="0.7142784" />
       <inertia
         ixx="0.00096626194"
@@ -86,57 +80,42 @@
         iyy="0.00575735994"
         iyz="-0.00039309867"
-        izz="0.00066079574" />
-    </inertial>
-    <visual>
-      <origin
-        xyz="0 0 0"
-        rpy="0 0 0" />
-      <geometry>
-        <mesh
-          filename="package://finalarm_simplified_description/meshes/link_2.STL" />
-      </geometry>
-      <material
-        name="">
-        <color
-          rgba="0.792156862745098 0.819607843137255 0.933333333333333 1" />
-      </material>
-    </visual>
-    <collision>
-      <origin
-        xyz="0 0 0"
-        rpy="0 0 0" />
-      <geometry>
-        <mesh
-          filename="package://finalarm_simplified_description/meshes/link_2.STL" />
-      </geometry>
-    </collision>
-  </link>
-  <joint
-    name="joint_1"
-    type="revolute">
-    <origin
-      xyz="0 0 0.0622"
-      rpy="3.1416 0 3.1416" />
-    <parent
-      link="base_link" />
-    <child
-      link="link_2" />
-    <axis
-      xyz="0 0 -1" />
-    <limit
-      lower="-3.14"
-      upper="3.14"
-      effort="6"
-      velocity="2" />
-    <dynamics damping="0.5"/>
-  </joint>
-  <link
-    name="link_3">
+        izz="0.00066079574"
+      />
+    </inertial>
+    <visual>
+      <origin xyz="0 0 0" rpy="0 0 0" />
+      <geometry>
+        <mesh
+          filename="package://finalarm_simplified_description/meshes/link_2.STL"
+        />
+      </geometry>
+      <material name="">
+        <color rgba="0.792156862745098 0.819607843137255 0.933333333333333 1" />
+      </material>
+    </visual>
+    <collision>
+      <origin xyz="0 0 0" rpy="0 0 0" />
+      <geometry>
+        <mesh
+          filename="package://finalarm_simplified_description/meshes/link_2.STL"
+        />
+      </geometry>
+    </collision>
+  </link>
+  <joint name="joint_1" type="revolute">
+    <origin xyz="0 0 0.0622" rpy="3.1416 0 3.1416" />
+    <parent link="base_link" />
+    <child link="link_2" />
+    <axis xyz="0 0 -1" />
+    <limit lower="-3.14" upper="3.14" effort="6" velocity="2" />
+    <dynamics damping="0.5" />
+  </joint>
+  <link name="link_3">
     <inertial>
       <origin
         xyz="0.00913796893535261 -0.110721113647521 0.000700000000000008"
-        rpy="0 0 0" />
-      <mass
-        value="0.26363602" />
+        rpy="0 0 0"
+      />
+      <mass value="0.26363602" />
       <inertia
         ixx="0.00067487030"
@@ -145,57 +124,39 @@
         iyy="0.00024791507"
         iyz="0.00002448920"
-        izz="0.000052259169" />
-    </inertial>
-    <visual>
-      <origin
-        xyz="0 0 0"
-        rpy="0 0 0" />
-      <geometry>
-        <mesh
-          filename="package://finalarm_simplified_description/meshes/link_3.STL" />
-      </geometry>
-      <material
-        name="">
-        <color
-          rgba="0.792156862745098 0.819607843137255 0.933333333333333 1" />
-      </material>
-    </visual>
-    <collision>
-      <origin
-        xyz="0 0 0"
-        rpy="0 0 0" />
-      <geometry>
-        <mesh
-          filename="package://finalarm_simplified_description/meshes/link_3.STL" />
-      </geometry>
-    </collision>
-  </link>
-  <joint
-    name="joint_2"
-    type="revolute">
-    <origin
-      xyz="0 0 -0.14225"
-      rpy="1.5708 0 0" />
-    <parent
-      link="link_2" />
-    <child
-      link="link_3" />
-    <axis
-      xyz="0 0 1" />
-    <limit
-      lower="-2.35"
-      upper="2.35"
-      effort="6"
-      velocity="2" />
-    <dynamics damping="0.5"/>
-  </joint>
-  <link
-    name="link_4">
-    <inertial>
-      <origin
-        xyz="0 -8.67361737988404E-19 -0.06225"
-        rpy="0 0 0" />
-      <mass
-        value="0.2302254" />
+        izz="0.000052259169"
+      />
+    </inertial>
+    <visual>
+      <origin xyz="0 0 0" rpy="0 0 0" />
+      <geometry>
+        <mesh
+          filename="package://finalarm_simplified_description/meshes/link_3.STL"
+        />
+      </geometry>
+      <material name="">
+        <color rgba="0.792156862745098 0.819607843137255 0.933333333333333 1" />
+      </material>
+    </visual>
+    <collision>
+      <origin xyz="0 0 0" rpy="0 0 0" />
+      <geometry>
+        <mesh
+          filename="package://finalarm_simplified_description/meshes/link_3.STL"
+        />
+      </geometry>
+    </collision>
+  </link>
+  <joint name="joint_2" type="revolute">
+    <origin xyz="0 0 -0.14225" rpy="1.5708 0 0" />
+    <parent link="link_2" />
+    <child link="link_3" />
+    <axis xyz="0 0 1" />
+    <limit lower="-2.35" upper="2.35" effort="6" velocity="2" />
+    <dynamics damping="0.5" />
+  </joint>
+  <link name="link_4">
+    <inertial>
+      <origin xyz="0 -8.67361737988404E-19 -0.06225" rpy="0 0 0" />
+      <mass value="0.2302254" />
       <inertia
         ixx="0.00012288342"
@@ -204,57 +165,42 @@
         iyy="0.00011093520"
         iyz="0.00000039768"
-        izz="0.00002956657" />
-    </inertial>
-    <visual>
-      <origin
-        xyz="0 0 0"
-        rpy="0 0 0" />
-      <geometry>
-        <mesh
-          filename="package://finalarm_simplified_description/meshes/link_4.STL" />
-      </geometry>
-      <material
-        name="">
-        <color
-          rgba="0.792156862745098 0.819607843137255 0.933333333333333 1" />
-      </material>
-    </visual>
-    <collision>
-      <origin
-        xyz="0 0 0"
-        rpy="0 0 0" />
-      <geometry>
-        <mesh
-          filename="package://finalarm_simplified_description/meshes/link_4.STL" />
-      </geometry>
-    </collision>
-  </link>
-  <joint
-    name="joint_3"
-    type="revolute">
-    <origin
-      xyz="0 -0.1721 0.0007"
-      rpy="-1.5708 0 0" />
-    <parent
-      link="link_3" />
-    <child
-      link="link_4" />
-    <axis
-      xyz="0 0 -1" />
-    <limit
-      lower="-3.14"
-      upper="3.14"
-      effort="6"
-      velocity="2" />
-    <dynamics damping="0.5"/>
-  </joint>
-  <link
-    name="link_5">
+        izz="0.00002956657"
+      />
+    </inertial>
+    <visual>
+      <origin xyz="0 0 0" rpy="0 0 0" />
+      <geometry>
+        <mesh
+          filename="package://finalarm_simplified_description/meshes/link_4.STL"
+        />
+      </geometry>
+      <material name="">
+        <color rgba="0.792156862745098 0.819607843137255 0.933333333333333 1" />
+      </material>
+    </visual>
+    <collision>
+      <origin xyz="0 0 0" rpy="0 0 0" />
+      <geometry>
+        <mesh
+          filename="package://finalarm_simplified_description/meshes/link_4.STL"
+        />
+      </geometry>
+    </collision>
+  </link>
+  <joint name="joint_3" type="revolute">
+    <origin xyz="0 -0.1721 0.0007" rpy="-1.5708 0 0" />
+    <parent link="link_3" />
+    <child link="link_4" />
+    <axis xyz="0 0 -1" />
+    <limit lower="-3.14" upper="3.14" effort="6" velocity="2" />
+    <dynamics damping="0.5" />
+  </joint>
+  <link name="link_5">
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